File: Hardware/Shield/Shield-0.6.brd (EAGLE design)
At the start: 85 x 56 mm, 45 parts, among them J2 M20X2, J6 Motors, Q1 BSS138, Q2 BSS138, U1 FDS4465, U2 FDS4465, U3 TPS62130RGTRQNF

Commit message: Shield Updates
Parts:
- removed FRAME1: FRAME-LETTERNO_PACKAGE, SparkFun-Aesthetics:DUMMY
Changed lines of the file:
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@@
 <grid distance="0.5" unitdist="mm" unit="mm" style="lines" multiple="1" display="yes" altdistance="0.05" altunitdist="mm" altunit="mm"/>
 <layers>
-<layer number="1" name="Top" color="4" fill="1" visible="no" active="yes"/>
+<layer number="1" name="Top" color="4" fill="1" visible="yes" active="yes"/>
 <layer number="16" name="Bottom" color="1" fill="1" visible="yes" active="yes"/>
 <layer number="17" name="Pads" color="2" fill="1" visible="yes" active="yes"/>
@@
 <attribute name="PROD_ID" value="DIO-11284" x="16.5" y="36.5" size="1.778" layer="28" rot="MR90" display="off"/>
 </element>
-<element name="FRAME1" library="SparkFun-Aesthetics" package="DUMMY" value="FRAME-LETTERNO_PACKAGE" x="-64.77" y="72.39">
-<attribute name="VERSION" value="v01" x="-64.77" y="72.39" size="1.778" layer="27" display="off"/>
-<attribute name="DESIGNER" value="Nobody" x="-64.77" y="72.39" size="1.778" layer="27" display="off"/>
-</element>
 <element name="H1" library="Robotois" package="STAND-OFF-PLATED" value="STAND-OFFPLATED" x="42.5" y="20"/>
