File: Hardware/Shield/Shield-0.6.sch (EAGLE design)
At the start: 45 parts, among them J2 M20X2, J6 Motors, Q1 BSS138, Q2 BSS138, U1 FDS4465, U2 FDS4465, U3 TPS62130RGTRQNF

Commit message: Shield Updates
Parts:
- removed FRAME1: FRAME-LETTERNO_PACKAGE, SparkFun-Aesthetics:FRAME-LETTERNO_PACKAGE
Other:
- note added: "Main Battery voltage for motors. Te buck converter provides the 5v power supply for the PI board and the modules."
- note added: "RJ Connectors, signal level shifters for I2C protection, utility buttons and power-indicative LEDs"
- note removed: "Connectors, signal level shifters (3.3v-5v), pull-up resistor for digital inputs and power-indicative LEDs"
- note removed: "Main Battery, buck converter that provides the 5v power supply for the PI board and the modules."
- moved on the sheet: J10, J2, J3, J4, J5, J6, J7, J8, J9, LED1, Q1, Q2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
